File: pcb/atreis.kicad_pcb (KiCad board)
At the start: 2 copper layers, 114 parts, among them SW1 SW_Push, U1 Elite-C

Commit message: Completed tracks and edge. Cleaned up drawings.
Parts:
- D1: renamed from D22; moved to B.Cu
- D10: renamed from D52; moved to B.Cu
- D11: renamed from D32; moved to B.Cu
- D12: renamed from D34; moved to B.Cu
- D13: renamed from D46; moved to B.Cu
- D14: renamed from D13; moved to B.Cu
- D15: renamed from D49; moved to B.Cu
- D16: renamed from D45; moved to B.Cu
- D17: renamed from D21; moved to B.Cu
- D18: renamed from D51; moved to B.Cu
- D19: renamed from D26; moved to B.Cu
- D2: renamed from D8; moved to B.Cu
- D20: renamed from D25; moved to B.Cu
- D21: renamed from D7; moved to B.Cu
- D22: renamed from D29; moved to B.Cu
- D23: renamed from D11; moved to B.Cu
- D24: renamed from D47; moved to B.Cu
- D25: renamed from D3; moved to B.Cu
- D26: renamed from D10; moved to B.Cu
- D27: renamed from D12; moved to B.Cu
- D28: renamed from D41; moved to B.Cu
- D29: renamed from D37; moved to B.Cu
- D3: renamed from D15; moved to B.Cu
- D30: renamed from D24; moved to B.Cu
- D31: renamed from D50; moved to B.Cu
- D32: renamed from D6; moved to B.Cu
- D33: renamed from D38; moved to B.Cu
- D34: renamed from D48; moved to B.Cu
- D35: renamed from D18; moved to B.Cu
- D36: renamed from D19; moved to B.Cu
- D37: renamed from D23; moved to B.Cu
- D38: renamed from D53; moved to B.Cu
- D39: renamed from D16; moved to B.Cu
- D4: renamed from D9; moved to B.Cu
- D40: renamed from D36; moved to B.Cu
- D41: renamed from D5; moved to B.Cu
- D42: renamed from D44; moved to B.Cu
- D43: renamed from D40; moved to B.Cu
- D44: renamed from D56; moved to B.Cu
- D45: renamed from D4; moved to B.Cu
- D46: renamed from D17; moved to B.Cu
- D47: renamed from D2; moved to B.Cu
- D48: renamed from D1; moved to B.Cu
- D49: renamed from D28; moved to B.Cu
- D5: renamed from D39; moved to B.Cu
- D50: renamed from D31; moved to B.Cu
- D51: renamed from D43; moved to B.Cu
- D52: renamed from D33; moved to B.Cu
- D53: renamed from D54; moved to B.Cu
- D54: renamed from D30; moved to B.Cu
- D55: renamed from D42; moved to B.Cu
- D56: renamed from D35; moved to B.Cu
- D6: renamed from D27; moved to B.Cu
- D7: renamed from D14; moved to B.Cu
- D8: renamed from D20; moved to B.Cu
- D9: renamed from D55; moved to B.Cu
- moved D46 501.4 mm to (310.4, 95.5), turned to -166.33 degrees
- moved U1 494.0 mm to (183.4, 105.9), turned to -90 degrees
- moved D52 493.5 mm to (311.0, 98.0), turned to -166.33 degrees
- moved D40 475.2 mm to (302.0, 60.9), turned to -166.33 degrees
- moved D51 474.3 mm to (292.5, 102.5), turned to -166.33 degrees
- moved D45 474.1 mm to (291.9, 100.0), turned to -166.33 degrees
- moved D33 445.9 mm to (282.9, 63.0), turned to -166.33 degrees
- moved D34 443.5 mm to (301.4, 58.5), turned to -166.33 degrees
- moved D50 442.6 mm to (272.8, 102.0), turned to -166.33 degrees
- moved D56 439.7 mm to (250.0, 129.8), turned to -166.33 degrees
- moved D39 434.5 mm to (283.5, 65.4), turned to -166.33 degrees
- moved D44 433.1 mm to (272.3, 99.8), turned to -166.33 degrees
- moved D49 423.0 mm to (253.6, 104.6), turned to -166.33 degrees
- moved D55 421.6 mm to (232.0, 136.5), turned to -166.33 degrees
- moved D37 416.5 mm to (244.8, 67.5), turned to -166.33 degrees
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- renumbered MX29 to MX1, MX45 to MX10, MX35 to MX11, MX1 to MX12, MX52 to MX13, MX6 to MX15, MX9 to MX16, MX55 to MX17, MX56 to MX18, MX47 to MX19, MX10 to MX2, MX41 to MX20, MX26 to MX22, MX44 to MX24, MX7 to MX25, MX34 to MX26, MX46 to MX27, MX4 to MX28, MX15 to MX29, MX54 to MX3, MX27 to MX30, MX16 to MX31, MX31 to MX32, MX18 to MX33, MX24 to MX34, MX49 to MX35, MX37 to MX36, MX17 to MX37, MX5 to MX38, MX38 to MX39, MX13 to MX4, MX32 to MX40, MX33 to MX41, MX50 to MX42, MX19 to MX43, MX39 to MX44, MX28 to MX45, MX22 to MX46, MX43 to MX47, MX42 to MX48, MX48 to MX49, MX30 to MX5, MX3 to MX50, MX53 to MX51, MX8 to MX52, MX40 to MX53, MX2 to MX54, MX25 to MX55, MX51 to MX56, MX11 to MX6, MX12 to MX7, MX36 to MX8, MX20 to MX9
Connections:
- D1 pad 1: ROW3 -> ROW0
- D1 pad 2: Net-(D22-Pad2) -> Net-(D1-Pad2)
- D10 pad 1: ROW6 -> ROW1
- D10 pad 2: Net-(D52-Pad2) -> Net-(D10-Pad2)
- D11 pad 1: ROW9 -> ROW1
- D11 pad 2: Net-(D32-Pad2) -> Net-(D11-Pad2)
- D12 pad 1: ROW9 -> ROW1
- D12 pad 2: Net-(D34-Pad2) -> Net-(D12-Pad2)
- D13 pad 1: ROW7 -> ROW2
- D13 pad 2: Net-(D46-Pad2) -> Net-(D13-Pad2)
- D14 pad 1: ROW2 -> ROW3
- D14 pad 2: Net-(D13-Pad2) -> Net-(D19-Pad2)
- D15 pad 1: ROW6 -> ROW2
- D15 pad 2: Net-(D49-Pad2) -> Net-(D14-Pad2)
- D16 pad 1: ROW7 -> ROW3
- D16 pad 2: Net-(D45-Pad2) -> Net-(D20-Pad2)
- D17 pad 1: ROW3 -> ROW2
- D17 pad 2: Net-(D21-Pad2) -> Net-(D15-Pad2)
- D18 pad 1: ROW6 -> ROW3
- D18 pad 2: Net-(D51-Pad2) -> Net-(D21-Pad2)
- D19 pad 1: ROW4 -> ROW2
- D19 pad 2: Net-(D26-Pad2) -> Net-(D16-Pad2)
- D2 pad 1: ROW1 -> ROW0
- D2 pad 2: Net-(D8-Pad2) -> Net-(D2-Pad2)
- D20 pad 1: ROW4 -> ROW3
- D20 pad 2: Net-(D25-Pad2) -> Net-(D22-Pad2)
- D21 pad 1: ROW1 -> ROW2
- D21 pad 2: Net-(D7-Pad2) -> Net-(D17-Pad2)
- D22 pad 1: ROW9 -> ROW3
- D22 pad 2: Net-(D29-Pad2) -> Net-(D23-Pad2)
- D23 pad 1: ROW1 -> ROW2
- D23 pad 2: Net-(D11-Pad2) -> Net-(D18-Pad2)
- D24 pad 1: ROW6 -> ROW3
- D24 pad 2: Net-(D47-Pad2) -> Net-(D24-Pad2)
- D25 pad 1: ROW0 -> ROW4
- D25 pad 2: Net-(D3-Pad2) -> Net-(D25-Pad2)
- D26 pad 1: ROW1 -> ROW4
- D26 pad 2: Net-(D10-Pad2) -> Net-(D26-Pad2)
- D27 pad 1: ROW1 -> ROW4
- D27 pad 2: Net-(D12-Pad2) -> Net-(D27-Pad2)
- D28 pad 1: ROW7 -> ROW4
- D28 pad 2: Net-(D41-Pad2) -> Net-(D28-Pad2)
- D29 pad 1: ROW8 -> ROW5
- D29 pad 2: Net-(D37-Pad2) -> Net-(D29-Pad2)
- D3 pad 1: ROW2 -> ROW0
- D3 pad 2: Net-(D15-Pad2) -> Net-(D3-Pad2)
- D30 pad 1: ROW3 -> ROW5
- D30 pad 2: Net-(D24-Pad2) -> Net-(D30-Pad2)
- D31 pad 1: ROW6 -> ROW5
- D31 pad 2: Net-(D50-Pad2) -> Net-(D31-Pad2)
- D32 pad 1: ROW0 -> ROW5
- D32 pad 2: Net-(D6-Pad2) -> Net-(D32-Pad2)
- D33 pad 1: ROW8 -> ROW5
- D33 pad 2: Net-(D38-Pad2) -> Net-(D33-Pad2)
- D34 pad 1: ROW6 -> ROW5
- D34 pad 2: Net-(D48-Pad2) -> Net-(D34-Pad2)
- D35 pad 1: ROW2 -> ROW6
- D35 pad 2: Net-(D18-Pad2) -> Net-(D35-Pad2)
- D36 pad 1: ROW3 -> ROW6
- D36 pad 2: Net-(D19-Pad2) -> Net-(D36-Pad2)
- D37 pad 1: ROW3 -> ROW6
- D37 pad 2: Net-(D23-Pad2) -> Net-(D37-Pad2)
- D38 pad 1: ROW5 -> ROW6
- D38 pad 2: Net-(D53-Pad2) -> Net-(D38-Pad2)
- D39 pad 1: ROW2 -> ROW6
- D39 pad 2: Net-(D16-Pad2) -> Net-(D39-Pad2)
- D4 pad 1: ROW1 -> ROW0
- D4 pad 2: Net-(D9-Pad2) -> Net-(D4-Pad2)
- D40 pad 1: ROW8 -> ROW6
- D40 pad 2: Net-(D36-Pad2) -> Net-(D40-Pad2)
- D41 pad 1: ROW0 -> ROW7
- D41 pad 2: Net-(D5-Pad2) -> Net-(D41-Pad2)
- D42 pad 2: Net-(D44-Pad2) -> Net-(D42-Pad2)
- D43 pad 1: ROW8 -> ROW7
- D43 pad 2: Net-(D40-Pad2) -> Net-(D43-Pad2)
- D44 pad 1: ROW5 -> ROW7
- D44 pad 2: Net-(D56-Pad2) -> Net-(D44-Pad2)
- D45 pad 1: ROW0 -> ROW7
- D45 pad 2: Net-(D4-Pad2) -> Net-(D45-Pad2)
- D46 pad 1: ROW2 -> ROW7
- D46 pad 2: Net-(D17-Pad2) -> Net-(D46-Pad2)
- D47 pad 1: ROW0 -> ROW8
- D47 pad 2: Net-(D2-Pad2) -> Net-(D47-Pad2)
- D48 pad 1: ROW0 -> ROW8
- D48 pad 2: Net-(D1-Pad2) -> Net-(D48-Pad2)
- D49 pad 1: ROW4 -> ROW8
- D49 pad 2: Net-(D28-Pad2) -> Net-(D49-Pad2)
- D5 pad 1: ROW8 -> ROW0
- D5 pad 2: Net-(D39-Pad2) -> Net-(D5-Pad2)
- D50 pad 1: ROW9 -> ROW8
- D50 pad 2: Net-(D31-Pad2) -> Net-(D50-Pad2)
- D51 pad 1: ROW7 -> ROW8
- D51 pad 2: Net-(D43-Pad2) -> Net-(D51-Pad2)
- D52 pad 1: ROW9 -> ROW8
- D52 pad 2: Net-(D33-Pad2) -> Net-(D52-Pad2)
- D53 pad 1: ROW5 -> ROW9
- D53 pad 2: Net-(D54-Pad2) -> Net-(D53-Pad2)
- D54 pad 2: Net-(D30-Pad2) -> Net-(D54-Pad2)
- D55 pad 1: ROW7 -> ROW9
- D55 pad 2: Net-(D42-Pad2) -> Net-(D55-Pad2)
- D56 pad 1: ROW8 -> ROW9
- D56 pad 2: Net-(D35-Pad2) -> Net-(D56-Pad2)
- D6 pad 1: ROW4 -> ROW0
- D6 pad 2: Net-(D27-Pad2) -> Net-(D6-Pad2)
- D7 pad 1: ROW2 -> ROW1
- D7 pad 2: Net-(D14-Pad2) -> Net-(D7-Pad2)
- D8 pad 1: ROW3 -> ROW1
- D8 pad 2: Net-(D20-Pad2) -> Net-(D8-Pad2)
- D9 pad 1: ROW5 -> ROW1
- D9 pad 2: Net-(D55-Pad2) -> Net-(D9-Pad2)
- MX1 pad 1: COL5 -> COL0
- MX1 pad 2: Net-(D29-Pad2) -> Net-(D1-Pad2)
- MX10 pad 1: COL1 -> COL3
- MX10 pad 2: Net-(D45-Pad2) -> Net-(D10-Pad2)
- MX11 pad 1: COL5 -> COL4
- MX11 pad 2: Net-(D35-Pad2) -> Net-(D11-Pad2)
- MX12 pad 1: COL0 -> COL5
- MX12 pad 2: Net-(D1-Pad2) -> Net-(D12-Pad2)
- MX13 pad 2: Net-(D52-Pad2) -> Net-(D13-Pad2)
- MX15 pad 1: COL5 -> COL2
- MX15 pad 2: Net-(D6-Pad2) -> Net-(D15-Pad2)
- MX16 pad 1: COL2 -> COL3
- MX16 pad 2: Net-(D9-Pad2) -> Net-(D16-Pad2)
- MX17 pad 1: COL3 -> COL4
- MX17 pad 2: Net-(D55-Pad2) -> Net-(D17-Pad2)
- MX18 pad 1: COL2 -> COL5
- MX18 pad 2: Net-(D56-Pad2) -> Net-(D18-Pad2)
- MX19 pad 1: COL5 -> COL0
- MX19 pad 2: Net-(D47-Pad2) -> Net-(D19-Pad2)
- MX2 pad 1: COL3 -> COL1
- MX2 pad 2: Net-(D10-Pad2) -> Net-(D2-Pad2)
- MX20 pad 1: COL5 -> COL1
- MX20 pad 2: Net-(D41-Pad2) -> Net-(D20-Pad2)
- MX22 pad 2: Net-(D26-Pad2) -> Net-(D22-Pad2)
- MX24 pad 1: COL2 -> COL5
- MX24 pad 2: Net-(D44-Pad2) -> Net-(D24-Pad2)
- MX25 pad 1: COL0 -> COL2
- MX25 pad 2: Net-(D7-Pad2) -> Net-(D25-Pad2)
- MX26 pad 1: COL0 -> COL3
- MX26 pad 2: Net-(D34-Pad2) -> Net-(D26-Pad2)
- MX27 pad 1: COL0 -> COL4
- MX27 pad 2: Net-(D46-Pad2) -> Net-(D27-Pad2)
- MX28 pad 1: COL3 -> COL5
- MX28 pad 2: Net-(D4-Pad2) -> Net-(D28-Pad2)
- MX29 pad 1: COL2 -> COL5
- MX29 pad 2: Net-(D15-Pad2) -> Net-(D29-Pad2)
- MX3 pad 1: COL4 -> COL2
- MX3 pad 2: Net-(D54-Pad2) -> Net-(D3-Pad2)
- MX30 pad 2: Net-(D27-Pad2) -> Net-(D30-Pad2)
- MX31 pad 2: Net-(D16-Pad2) -> Net-(D31-Pad2)
- MX32 pad 1: COL3 -> COL2
- MX32 pad 2: Net-(D31-Pad2) -> Net-(D32-Pad2)
- MX33 pad 1: COL5 -> COL1
- MX33 pad 2: Net-(D18-Pad2) -> Net-(D33-Pad2)
- MX34 pad 1: COL5 -> COL0
- MX34 pad 2: Net-(D24-Pad2) -> Net-(D34-Pad2)
- MX35 pad 1: COL3 -> COL5
- MX35 pad 2: Net-(D49-Pad2) -> Net-(D35-Pad2)
- MX36 pad 1: COL3 -> COL4
- MX36 pad 2: Net-(D37-Pad2) -> Net-(D36-Pad2)
- MX37 pad 1: COL4 -> COL3
- MX37 pad 2: Net-(D17-Pad2) -> Net-(D37-Pad2)
- MX38 pad 1: COL4 -> COL2
- MX38 pad 2: Net-(D5-Pad2) -> Net-(D38-Pad2)
- MX39 pad 1: COL2 -> COL1
- MX39 pad 2: Net-(D38-Pad2) -> Net-(D39-Pad2)
- MX4 pad 1: COL0 -> COL3
- MX4 pad 2: Net-(D13-Pad2) -> Net-(D4-Pad2)
- MX40 pad 1: COL2 -> COL0
- MX40 pad 2: Net-(D32-Pad2) -> Net-(D40-Pad2)
- MX41 pad 1: COL1 -> COL5
- MX41 pad 2: Net-(D33-Pad2) -> Net-(D41-Pad2)
- MX42 pad 1: COL2 -> COL4
- MX42 pad 2: Net-(D50-Pad2) -> Net-(D42-Pad2)
- MX43 pad 1: COL0 -> COL3
- MX43 pad 2: Net-(D19-Pad2) -> Net-(D43-Pad2)
- MX44 pad 1: COL1 -> COL2
- MX44 pad 2: Net-(D39-Pad2) -> Net-(D44-Pad2)
- MX45 pad 1: COL5 -> COL1
- MX45 pad 2: Net-(D28-Pad2) -> Net-(D45-Pad2)
- MX46 pad 1: COL3 -> COL0
- MX46 pad 2: Net-(D22-Pad2) -> Net-(D46-Pad2)
- MX47 pad 1: COL3 -> COL5
- MX47 pad 2: Net-(D43-Pad2) -> Net-(D47-Pad2)
- MX48 pad 2: Net-(D42-Pad2) -> Net-(D48-Pad2)
- MX49 pad 1: COL4 -> COL3
- MX49 pad 2: Net-(D48-Pad2) -> Net-(D49-Pad2)
- MX5 pad 2: Net-(D30-Pad2) -> Net-(D5-Pad2)
- MX50 pad 2: Net-(D3-Pad2) -> Net-(D50-Pad2)
- MX51 pad 1: COL5 -> COL1
- MX51 pad 2: Net-(D53-Pad2) -> Net-(D51-Pad2)
- MX52 pad 1: COL1 -> COL0
- MX52 pad 2: Net-(D8-Pad2) -> Net-(D52-Pad2)
- MX53 pad 1: COL0 -> COL5
- MX53 pad 2: Net-(D40-Pad2) -> Net-(D53-Pad2)
- MX54 pad 1: COL1 -> COL4
- MX54 pad 2: Net-(D2-Pad2) -> Net-(D54-Pad2)
- MX55 pad 1: COL2 -> COL3
- MX55 pad 2: Net-(D25-Pad2) -> Net-(D55-Pad2)
- MX56 pad 1: COL1 -> COL2
- MX56 pad 2: Net-(D51-Pad2) -> Net-(D56-Pad2)
- MX6 pad 1: COL4 -> COL5
- MX6 pad 2: Net-(D11-Pad2) -> Net-(D6-Pad2)
- MX7 pad 1: COL5 -> COL0
- MX7 pad 2: Net-(D12-Pad2) -> Net-(D7-Pad2)
- MX8 pad 1: COL4 -> COL1
- MX8 pad 2: Net-(D36-Pad2) -> Net-(D8-Pad2)
- MX9 pad 1: COL1 -> COL2
- MX9 pad 2: Net-(D20-Pad2) -> Net-(D9-Pad2)
- U1 pad 13: ROW5 -> ROW9
- U1 pad 14: ROW6 -> ROW8
- U1 pad 16: ROW8 -> ROW6
- U1 pad 17: ROW9 -> ROW5
- U1 pad 23: unconnected-(U1-Pad23) -> GND
- U1 pad 3: unconnected-(U1-Pad3) -> GND
- U1 pad 4: unconnected-(U1-Pad4) -> GND
Routing:
- net COL2: track 0.00 -> 385.9 mm, vias 0 -> 1
- net COL0: track 0.00 -> 378.7 mm, vias 0 -> 1
- net COL3: track 0.00 -> 347.6 mm, vias 0 -> 1
- net COL1: track 0.00 -> 343.9 mm, vias 0 -> 1
- net COL4: track 0.00 -> 324.0 mm, vias 0 -> 1
- net COL5: track 0.00 -> 245.3 mm, vias 0 -> 1
- net ROW5: track 0.00 -> 145.1 mm
- net ROW6: track 0.00 -> 143.3 mm
- net ROW1: track 0.00 -> 133.7 mm
- net ROW0: track 0.00 -> 133.4 mm
- net ROW8: track 0.00 -> 130.4 mm
- net ROW7: track 0.00 -> 129.4 mm
- net ROW3: track 0.00 -> 119.6 mm
- net ROW2: track 0.00 -> 119.0 mm
- net ROW9: track 0.00 -> 79.4 mm
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Other:
- board outline added: 284 x 140.8 mm

Commit message: Updated tracks that were too close to the holes.
Routing:
- net COL1: track 343.9 -> 344.7 mm
- net COL0: track 378.7 -> 379.4 mm
- net COL2: track 385.9 -> 386.5 mm
Other:
- outline, holes or cut-outs redrawn
