File: pcb/atreis.kicad_pcb (KiCad board)
At the start: 2 copper layers, 284 x 140.8 mm, 114 parts, among them SW1 SW_Push, U1 Elite-C

Commit message: Added bottom side of the case. Rerouted some tracks to make space for the holes in the middle of the PCB. Added holes to the top case.
Routing:
- net ROW1: track 133.7 -> 134.8 mm
- net ROW3: track 119.6 -> 120.7 mm
Other:
- outline, holes or cut-outs redrawn

Commit message: Rerouted some of the tracks. Much nicer now. Rerouted tracks to make the holes thru holes, to use with spacers. Re-generated gerber file.
Parts:
- added ?: , , F.Cu at (71.0, 100.5)
- added REF**: M2_Hole_NPTH_Outside, kbd:M2_Hole_NPTH_Outside, F.Cu at (120.4, 41.1)
- added REF**: M2_Hole_NPTH_Outside, kbd:M2_Hole_NPTH_Outside, F.Cu at (211.9, 77.9)
- added REF**: M2_Hole_NPTH_Outside, kbd:M2_Hole_NPTH_Outside, F.Cu at (295.7, 100.5)
- added REF**: M2_Hole_NPTH_Outside, kbd:M2_Hole_NPTH_Outside, F.Cu at (286.8, 63.5)
- added REF**: M2_Hole_NPTH_Outside, kbd:M2_Hole_NPTH_Outside, F.Cu at (45.5, 116.1)
- added REF**: M2_Hole_NPTH_Outside, kbd:M2_Hole_NPTH_Outside, F.Cu at (105.0, 149.9)
- added REF**: M2_Hole_NPTH_Outside, kbd:M2_Hole_NPTH_Outside, F.Cu at (154.9, 77.9)
- added REF**: M2_Hole_NPTH_Outside, kbd:M2_Hole_NPTH_Outside, F.Cu at (246.3, 41.1)
- added REF**: M2_Hole_NPTH_Outside, kbd:M2_Hole_NPTH_Outside, F.Cu at (155.8, 144.9)
- added REF**: M2_Hole_NPTH_Outside, kbd:M2_Hole_NPTH_Outside, F.Cu at (145.9, 115.0)
- added REF**: M2_Hole_NPTH_Outside, kbd:M2_Hole_NPTH_Outside, F.Cu at (161.0, 56.2)
- added REF**: M2_Hole_NPTH_Outside, kbd:M2_Hole_NPTH_Outside, F.Cu at (201.2, 167.5)
- added REF**: M2_Hole_NPTH_Outside, kbd:M2_Hole_NPTH_Outside, F.Cu at (205.8, 56.2)
- added REF**: M2_Hole_NPTH_Outside, kbd:M2_Hole_NPTH_Outside, F.Cu at (165.6, 167.5)
- added REF**: M2_Hole_NPTH_Outside, kbd:M2_Hole_NPTH_Outside, F.Cu at (210.9, 144.9)
- added REF**: M2_Hole_NPTH_Outside, kbd:M2_Hole_NPTH_Outside, F.Cu at (80.0, 63.5)
- added REF**: M2_Hole_NPTH_Outside, kbd:M2_Hole_NPTH_Outside, F.Cu at (321.3, 116.1)
- added REF**: M2_Hole_NPTH_Outside, kbd:M2_Hole_NPTH_Outside, F.Cu at (302.6, 38.0)
- added REF**: M2_Hole_NPTH_Outside, kbd:M2_Hole_NPTH_Outside, F.Cu at (64.2, 38.0)
- added REF**: M2_Hole_NPTH_Outside, kbd:M2_Hole_NPTH_Outside, F.Cu at (261.8, 149.9)
- added REF**: M2_Hole_NPTH_Outside, kbd:M2_Hole_NPTH_Outside, F.Cu at (220.8, 115.0)
- moved D28 0.69 mm to (161.3, 142.6)
- moved D27 0.51 mm to (155.9, 148.5)
- moved D53 0.46 mm to (212.0, 141.0)
- moved D54 0.41 mm to (217.0, 147.1)
Routing:
- net COL5: track 245.3 -> 212.5 mm
- net COL2: track 386.5 -> 391.3 mm
- net COL4: track 324.3 -> 326.0 mm
- net COL0: track 379.4 -> 380.5 mm
- net COL1: track 344.7 -> 345.7 mm
- net COL3: track 347.2 -> 347.8 mm
- net Net-(D28-Pad2): track 20.6 -> 20.0 mm
- net Net-(D53-Pad2): track 6.67 -> 7.18 mm
Other:
- outline, holes or cut-outs redrawn
